File: voltage ref calibration tool.kicad_pcb (KiCad board)
At the start: 2 copper layers, 147.1 x 79.5 mm, 70 parts, among them J1 AudioJack2_SwitchT, J2 Molex-MicroFit_43650-0316, J3 AudioJack2_SwitchT, J4 Conn_01x02, J5 Conn_01x02, SW1 SW_SP6T, SW2 B3F-1020, SW3 B3F-1020, SW4 B3F-1020, SW5 B3F-1020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

Commit message: Add copyright legend to schematic and pcb.
Other:
- board text added: "May 2024"
- board text added: "© 2024 by Aaron Kimball Licensed under CC BY-SA 4.0. https://creativecommons.org/licenses/by-sa/4.0/"
Changed lines of the file:
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@@
+		)
+	)
+	(gr_text "© 2024 by Aaron Kimball\nLicensed under CC BY-SA 4.0.\nhttps://creativecommons.org/licenses/by-sa/4.0/"
+		(at 179.832 179.578 0)
+		(layer "Dwgs.User")
+		(effects
+			(font
+				(size 1 1)
+				(thickness 0.15)
+			)
+			(justify left bottom)
+		)
+	)
+	(gr_text "May 2024"
+		(at 206.121 193.167 0)
+		(layer "Dwgs.User")
+		(effects
+			(font
+				(size 1 1)
+				(thickness 0.15)
+			)
+			(justify left bottom)
 		)
 	)
 	(gr_text "PRECISION VOLTAGE REFERENCE CALIBRATION TOOL\n"
-		(at 231.394 174.244 0)
+		(at 229.235 168.529 0)
 		(layer "Dwgs.User")
 		(effects
